File: hardware/kicad/panel-keyboard/panel-keyboard.kicad_sch (KiCad schematic)
At the start: 113 parts, among them J2 SWD_1.27, J485 2EDGVC-5.08-03P, Q12 AO4407A, SW1 Tact_12mm, SW10 Tact_12mm, SW11 Tact_12mm, SW12 Tact_12mm, SW13 Tact_12mm, SW14 Tact_12mm, SW15 Tact_12mm, SW16 Tact_12mm, SW2 Tact_12mm, SW3 Tact_12mm, SW4 Tact_12mm, SW5 Tact_12mm, SW6 Tact_12mm, SW7 Tact_12mm, SW8 Tact_12mm, SW9 Tact_12mm, U1 STM32F030F4P6, U2 TM1638, U3 MAX485CSA, U4 XL1509-5.0, U5 AMS1117-3.3

Commit message: update layout và chip để mạch thành dạng hình vuông 120x120mm
Parts:
- removed C14, C21, CC1, CC2, CC3, CC4, CK1, CK2, CK3, CK4: 100nF, Capacitor_SMD:C_0805_2012Metric, symbol Device:C
- removed CTM1: 100n, Capacitor_SMD:C_0805_2012Metric, symbol Device:C
- removed CTM2: 10u, Capacitor_SMD:C_0805_2012Metric, symbol Device:C
- removed CVDDA: 1uF, Capacitor_SMD:C_0805_2012Metric, symbol Device:C
- removed FB1, FB2, FB5V: BLM21PG121, Inductor_SMD:L_0805_2012Metric, symbol Device:Ferrite_Bead
- removed Q12: AO4407A, Package_TO_SOT_SMD:SOT-23, symbol Transistor_FET:Q_PMOS_GSD
- removed R33A, R33B, R33C: 33, Resistor_SMD:R_0805_2012Metric, symbol Device:R
- removed RBOT0: 10k, Resistor_SMD:R_0805_2012Metric, symbol Device:R
- removed RLED1, RLED2, RLED3, RLED4, RLED5, RLED6, RLED7, RLED8: 1k, Resistor_SMD:R_0805_2012Metric, symbol Device:R
- removed RPU: 4.7k, Resistor_SMD:R_0805_2012Metric, symbol Device:R
- removed U1: STM32F030F4P6, Package_SO:TSSOP-20_4.4x6.5mm_P0.65mm, symbol MCU_ST_STM32F0:STM32F030F4Px
- removed U2: TM1638, Panel:SOIC-28_TM1638, symbol Panel:TM1638
- added CLED: 100n, Capacitor_SMD:C_0805_2012Metric, symbol Device:C
- added FB1, FB2, FB5V: BLM21PG121, Inductor_SMD:L_0805_2012Metric, symbol Device:FerriteBead
- added Q17: AO4407A, Package_TO_SOT_SMD:SOT-23, symbol Transistor_FET:Q_PMOS_GSD
- added RPK1, RPK2, RPK3, RPK4: 10k, Resistor_SMD:R_0805_2012Metric, symbol Device:R
- added RSCL, RSDA: 4.7k, Resistor_SMD:R_0805_2012Metric, symbol Device:R
- added U1: STM32G030C8T6, Package_QFP:LQFP-48_7x7mm_P0.5mm, symbol MCU_ST_STM32G0:STM32G030C8Tx
- added U6: HT16K33A, Panel:HT16K33A_SSOP28, symbol Panel:HT16K33A
Connections:
- no-connect marks 7 -> 35
Other:
- title: Panel Keyboard All-in-One 100x150 -> Panel Keyboard All-in-One 120x120

Commit message: sửa danh sách linh kiện theo hương thương mại và add firmware cơ bản cho modbus
Parts:
- removed CLED: 100n, Capacitor_SMD:C_0805_2012Metric, symbol Device:C
- removed DS1, DS2, DS3, DS4, DS5, DS6, DS7, DS8: 7SEG_0.56_CC, Panel:LED7seg_1digit_0.56in_CC_THT, symbol Connector_Generic:Conn_01x10
- removed L2, L485: ACM2012-201, Inductor_SMD:L_CommonModeChoke_Coilank_ACM2012, symbol Device:Filter_EMI_CommonMode
- removed Q17: AO4407A, Package_TO_SOT_SMD:SOT-23, symbol Transistor_FET:Q_PMOS_GSD
- removed R17: 100k, Resistor_SMD:R_0805_2012Metric, symbol Device:R
- removed R36: 3k, Resistor_SMD:R_0805_2012Metric, symbol Device:R
- removed R37: 1k, Resistor_SMD:R_0805_2012Metric, symbol Device:R
- removed R38, RNST, RPK1, RPK2, RPK3, RPK4: 10k, Resistor_SMD:R_0805_2012Metric, symbol Device:R
- removed RC1, RC2, RC3, RC4, RK1, RK2, RK3, RK4: 100, Resistor_SMD:R_0805_2012Metric, symbol Device:R
- removed RSCL, RSDA: 4.7k, Resistor_SMD:R_0805_2012Metric, symbol Device:R
- removed RV1: 14D390K, Varistor:Varistor_Panasonic_VF, symbol Device:Varistor
- removed U1: STM32G030C8T6, Package_QFP:LQFP-48_7x7mm_P0.5mm, symbol MCU_ST_STM32G0:STM32G030C8Tx
- removed U6: HT16K33A, Panel:HT16K33A_SSOP28, symbol Panel:HT16K33A
- added BZ1: Active buzzer 5V 12x9.5, Buzzer_Beeper:Buzzer_12x9.5RM7.6, symbol Device:Buzzer
- added CLED1, CLED2: 100nF, Capacitor_SMD:C_0805_2012Metric, symbol Device:C
- added CLED3: 10uF, Capacitor_SMD:C_0805_2012Metric, symbol Device:C
- added DREV: SS34, Diode_SMD:D_SMA, symbol Device:D
- added DS1, DS2: 5641AS (4 digit 0.56in CC), Panel:Display_4digit_0.56in_THT, symbol Connector_Generic:Conn_01x12
- added FBIN: 600R@100MHz 2A, Inductor_SMD:L_0805_2012Metric, symbol Device:FerriteBead
- added QBZ: 2N7002, Package_TO_SOT_SMD:SOT-23, symbol Transistor_FET:2N7002
- added RBZG: 100k, Resistor_SMD:R_0805_2012Metric, symbol Device:R
- added RCLK, RDIO, RSTB: 4.7k, Resistor_SMD:R_0805_2012Metric, symbol Device:R
- added U1: STM32G030F6P6, Package_SO:TSSOP-20_4.4x6.5mm_P0.65mm, symbol MCU_ST_STM32G0:STM32G030F6Px
- added U6: TM1638, Package_SO:SOIC-28W_7.5x17.9mm_P1.27mm, symbol Panel:TM1638
- C15, C17: value 100nF -> 100nF 50V
- C16, C19: value 10uF -> 10uF 50V; footprint Capacitor_SMD:C_0805_2012Metric -> Capacitor_SMD:C_1206_3216Metric
- C2, C22: value 220uF -> 220uF 10V
- C4: value 1000uF -> 470uF 35V; footprint Capacitor_SMD:CP_Elec_10x12.5 -> Capacitor_SMD:CP_Elec_10x10.5
- CM3, CNRST, CVDD1: value 100n -> 100nF
- D8: footprint Diode_SMD:D_SOD-123 -> Diode_SMD:D_SMA
- F1: value MF-MSMF350 -> PPTC 1812 0.5A 33V; footprint Fuse:Fuse_2920_7451Metric -> Fuse:Fuse_1812_4532Metric
- FB1, FB2, FB5V: value BLM21PG121 -> 120R@100MHz 2A
- J2: value SWD_1.27 -> SWD (DNP); footprint Connector_PinHeader_1.27mm:PinHeader_1x04_P1.27mm_Vertical -> Connector_PinHeader_2.54mm:PinHeader_1x04_P2.54mm_Vertical
- J485: value 2EDGVC-5.08-03P -> KF2EDGV-5.08-3P
- J_PWR: value 2EDGVC-5.08-02P -> KF2EDGV-5.08-2P
- L1: value 47uH -> 47uH 6045; footprint Inductor_SMD:L_1210_3225Metric -> Inductor_SMD:L_Taiyo-Yuden_NR-60xx
- U3: value MAX485CSA -> SIT3485 / MAX3485
- U4: value XL1509-5.0 -> XL1509-5.0E1; footprint Package_TO_SOT_SMD:TO-263-5_TabPin3 -> Package_SO:SOIC-8_3.9x4.9mm_P1.27mm
Connections:
- no-connect marks 35 -> 10

Commit message: tạo c# app, update firmware để bàn phím hỗ trợ cả 2 mode slave/master. hỗ trợ giắc nạp và debug trên board phù hợp với mạch nạp DAPLINK STM32 cổng Type-C
Parts:
- removed J2: SWD (DNP), Connector_PinHeader_2.54mm:PinHeader_1x04_P2.54mm_Vertical, symbol Connector_Generic:Conn_01x04
- removed U3: SIT3485 / MAX3485, Package_SO:SOIC-8_3.9x4.9mm_P1.27mm, symbol Interface_UART:MAX485E
- added J_KEY: Membrane 1x10 2.54, Panel:Membrane_1x10_P2.54_Vertical_Slot, symbol Connector_Generic:Conn_01x10
- added J_LOG: DAP COM (DNP), Connector_PinHeader_2.54mm:PinHeader_1x04_P2.54mm_Vertical, symbol Connector_Generic:Conn_01x04
- added J_SWD: DAP SWD (DNP), Connector_PinHeader_2.54mm:PinHeader_1x04_P2.54mm_Vertical, symbol Connector_Generic:Conn_01x04
- added U3: SP3485EN, Package_SO:SOIC-8_3.9x4.9mm_P1.27mm, symbol Interface_UART:SP3485EN
- C16, C19: value 10uF 50V -> 2.2uF 50V X7R
- C2, C22: value 220uF 10V -> 220uF 10V RVT1A221M0605
- C4: value 470uF 35V -> 470uF 35V RVT1V471M1010
- F1: value PPTC 1812 0.5A 33V -> mSMD050-33V (PPTC 0.5A 33V)
- FB1, FB2, FB5V: value 120R@100MHz 2A -> GZ2012D101TF 100R
- FBIN: value 600R@100MHz 2A -> GZ2012D601TF 600R
- J485: value KF2EDGV-5.08-3P -> KF301-5.08-3P
- J_PWR: value KF2EDGV-5.08-2P -> KF301-5.08-2P
- L1: value 47uH 6045 -> SWPA6045S470MT 47uH
- SW1, SW10, SW11, SW12, SW13, SW14, SW15, SW16, SW2, SW3, SW4, SW5, SW6, SW7, SW8, SW9: value Tact_12mm -> B3F-4055
- TVS1: value SMAJ28A -> SMAJ28CA
- TVS2: value SM712 -> PSM712-LF-T7
Connections:
- no-connect marks 10 -> 8
